File: Schematic dan Board Project PT PETROKIMIA GRESIK/LCD 16x2 + PIN Button.brd (EAGLE design)
At the start: 95.2 x 58.1 mm, 5 parts

Commit message: Menambahkan File Project dan PDF untuk di print
Parts:
- moved X3 4.02 mm to (81.3, 52.1), turned to 270 degrees
Routing:
- net GND: track 72.1 -> 75.7 mm
Other:
- board text added: "Object Counting"
- board text added: "Tondi dan Goldi"
Changed lines of the file:
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@@
 <grid distance="50" unitdist="mil" unit="mil" style="lines" multiple="1" display="no" altdistance="5" altunitdist="mil" altunit="mil"/>
 <layers>
-<layer number="1" name="Top" color="4" fill="1" visible="yes" active="yes"/>
+<layer number="1" name="Top" color="4" fill="1" visible="no" active="yes"/>
 <layer number="2" name="Route2" color="16" fill="1" visible="no" active="no"/>
 <layer number="3" name="Route3" color="17" fill="1" visible="no" active="no"/>
@@
 <layer number="18" name="Vias" color="2" fill="1" visible="yes" active="yes"/>
 <layer number="19" name="Unrouted" color="6" fill="1" visible="yes" active="yes"/>
-<layer number="20" name="Dimension" color="24" fill="1" visible="yes" active="yes"/>
+<layer number="20" name="Dimension" color="24" fill="1" visible="no" active="yes"/>
 <layer number="21" name="tPlace" color="7" fill="1" visible="no" active="yes"/>
 <layer number="22" name="bPlace" color="7" fill="1" visible="yes" active="yes"/>
@@
 <dimension x1="16.51" y1="72.39" x2="85.09" y2="72.39" x3="50.8" y3="74.93" textsize="1.778" layer="1" visible="yes"/>
 <dimension x1="88.9" y1="67.31" x2="88.9" y2="45.72" x3="91.44" y3="56.515" textsize="1.778" layer="1" visible="yes"/>
+<text x="35.56" y="63.5" size="1.778" layer="16" rot="MR0">Object Counting</text>
+<text x="35.56" y="59.69" size="1.778" layer="16" rot="MR0">Tondi dan Goldi</text>
 </plain>
 <attributes>
@@
 <attribute name="VALUE" x="41.8338" y="60.325" size="1.778" layer="27" ratio="10" rot="R180"/>
 </element>
-<element name="X3" library="con-ptr500" library_urn="urn:adsk.eagle:library:181" package="AK500/2-H" package3d_urn="urn:adsk.eagle:package:9901/1" value="" x="77.47" y="53.34" smashed="yes" rot="R90">
-<attribute name="MF" value="" x="77.47" y="53.34" size="1.778" layer="27" rot="R90" display="off"/>
-<attribute name="MPN" value="" x="77.47" y="53.34" size="1.778" layer="27" rot="R90" display="off"/>
-<attribute name="NAME" x="73.914" y="48.26" size="1.778" layer="25" ratio="10" rot="R90"/>
-<attribute name="OC_FARNELL" value="unknown" x="77.47" y="53.34" size="1.778" layer="27" rot="R90" display="off"/>
-<attribute name="OC_NEWARK" value="unknown" x="77.47" y="53.34" size="1.778" layer="27" rot="R90" display="off"/>
-<attribute name="POPULARITY" value="3" x="77.47" y="53.34" size="1.778" layer="27" rot="R90" display="off"/>
-<attribute name="VALUE" x="86.995" y="48.26" size="1.778" layer="27" ratio="10" rot="R90"/>
+<element name="X3" library="con-ptr500" library_urn="urn:adsk.eagle:library:181" package="AK500/2-H" package3d_urn="urn:adsk.eagle:package:9901/1" value="" x="81.28" y="52.07" smashed="yes" rot="R270">
+<attribute name="MF" value="" x="81.28" y="52.07" size="1.778" layer="27" rot="R270" display="off"/>
+<attribute name="MPN" value="" x="81.28" y="52.07" size="1.778" layer="27" rot="R270" display="off"/>
+<attribute name="NAME" x="84.836" y="57.15" size="1.778" layer="25" ratio="10" rot="R270"/>
+<attribute name="OC_FARNELL" value="unknown" x="81.28" y="52.07" size="1.778" layer="27" rot="R270" display="off"/>
+<attribute name="OC_NEWARK" value="unknown" x="81.28" y="52.07" size="1.778" layer="27" rot="R270" display="off"/>
+<attribute name="POPULARITY" value="3" x="81.28" y="52.07" size="1.778" layer="27" rot="R270" display="off"/>
+<attribute name="VALUE" x="71.755" y="57.15" size="1.778" layer="27" ratio="10" rot="R270"/>
 </element>
 </elements>
@@
 <wire x1="39.88" y1="64.77" x2="72.39" y2="64.77" width="0.4064" layer="16"/>
 <wire x1="72.39" y1="64.77" x2="75.18" y2="61.98" width="0.4064" layer="16"/>
-<wire x1="77.4446" y1="50.8" x2="77.47" y2="50.8254" width="0.4064" layer="16"/>
 <wire x1="60.8584" y1="50.8" x2="68.58" y2="50.8" width="0.4064" layer="16"/>
 <wire x1="68.58" y1="50.8" x2="74.93" y2="50.8" width="0.4064" layer="16"/>
-<wire x1="74.93" y1="50.8" x2="77.4446" y2="50.8" width="0.4064" layer="16"/>
 <wire x1="68.58" y1="54.61" x2="68.58" y2="50.8" width="0.4064" layer="16"/>
 <wire x1="75.18" y1="61.97" x2="75.18" y2="56.45901875" width="0.4064" layer="16"/>
 <wire x1="75.18" y1="56.45901875" x2="75.1332" y2="56.41221875" width="0.4064" layer="16"/>
 <wire x1="75.1332" y1="51.0032" x2="74.93" y2="50.8" width="0.4064" layer="16"/>
-<wire x1="75.1332" y1="56.41221875" x2="75.1332" y2="51.0032" width="0.4064" layer="16"/>
+<wire x1="75.1332" y1="56.41221875" x2="75.1332" y2="54.61" width="0.4064" layer="16"/>
+<wire x1="75.1332" y1="54.61" x2="75.1332" y2="51.0032" width="0.4064" layer="16"/>
+<wire x1="81.28" y1="54.5846" x2="75.1586" y2="54.5846" width="0.4064" layer="16"/>
+<wire x1="75.1586" y1="54.5846" x2="75.1332" y2="54.61" width="0.4064" layer="16"/>
 </signal>
 <signal name="VCC">
